Commit message: Refactor urdf inertials and materials.
1. Adapt the urdf for inertials and materials from the robot description for curio.

File: rs750_description/urdf/rs750.urdf.xacro (robot description, xacro)
@@ -1,154 +1,171 @@
 <?xml version="1.0" ?>
-<robot name="bbot" xmlns:xacro="http://www.ros.org/wiki/xacro">
-  <!-- Math constants -->
-  <xacro:property name="math_pi" value="3.141592653589793" />
-  <!-- Math macros -->
-  <xacro:macro name="box_inertial" params="mass x y z">
-    <inertial>
-      <mass value="${mass}" />
-      <inertia
-        ixx="${mass * (y * y + z * z) / 12.0}" ixy="0.0" ixz="0.0"
-        iyy="${mass * (z * z + x * x) / 12.0}" iyz="0.0"
-        izz="${mass * (x * x + y * y) / 12.0}" />
-    </inertial>
-  </xacro:macro>
-  <!-- Constants for robot dimensions -->
-  <xacro:property name="hull_mass" value="20000.0" />
-  <xacro:property name="hull_loa" value="10.0" />
-  <xacro:property name="hull_woa" value="4.0" />
-  <xacro:property name="hull_doa" value="2.0" />
-  <xacro:property name="cam_mass" value="0.1" />
-  <xacro:property name="cam_size" value="0.1" />
-  <xacro:property name="ray_mass" value="0.1" />
-  <xacro:property name="ray_size" value="0.1" />
-  <xacro:property name="imu_mass" value="0.1" />
-  <xacro:property name="imu_size" value="0.1" />
-  <xacro:property name="gps_mass" value="0.1" />
-  <xacro:property name="gps_size" value="0.1" />
-  <xacro:property name="mag_mass" value="0.1" />
-  <xacro:property name="mag_size" value="0.1" />
-  <!-- Import Gazebo elements -->
-  <xacro:include filename="$(find bbot_description)/urdf/bbot.gazebo" />
-  <!-- Import materials -->
-  <xacro:include filename="$(find bbot_description)/urdf/materials.xacro" />
-  <!-- Base link (main hull) -->
-  <link name="base_link">
-    <visual>
-      <geometry>
-        <box size="${hull_loa} ${hull_woa} ${hull_doa}"/>
-      </geometry>
-      <material name="orange" />
-    </visual>
-    <collision>
-      <geometry>
-        <box size="${hull_loa} ${hull_woa} ${hull_doa}"/>
-      </geometry>
-    </collision>
-    <xacro:box_inertial mass="${hull_mass}" x="${hull_loa}" y="${hull_loa}" z="${hull_doa}" />
-  </link>
-  <!-- Camera -->
-  <link name="cam_link">
-    <visual>
-      <geometry>
-        <box size="${cam_size} ${cam_size} ${cam_size}"/>
-      </geometry>
-      <material name="red" />
-    </visual>
-    <collision>
-      <geometry>
-        <box size="${cam_size} ${cam_size} ${cam_size}"/>
-      </geometry>
-    </collision>
-    <xacro:box_inertial mass="${cam_mass}" x="${cam_size}" y="${cam_size}" z="${cam_size}" />
-  </link>
-  <joint name="cam_joint" type="fixed">
-    <axis xyz="0 1 0" />
-    <origin xyz="${hull_loa/2 - 0.25} 0 ${hull_doa/2 + cam_size/2}" rpy="0 0 0"/>
-    <parent link="base_link"/>
-    <child link="cam_link"/>
-  </joint>
-  <!-- Ray -->
-  <link name="ray_link">
-    <visual>
-      <geometry>
-        <box size="${ray_size} ${ray_size} ${ray_size}"/>
-      </geometry>
-      <material name="red" />
-    </visual>
-    <collision>
-      <geometry>
-        <box size="${ray_size} ${ray_size} ${ray_size}"/>
-      </geometry>
-    </collision>
-    <xacro:box_inertial mass="${ray_mass}" x="${ray_size}" y="${ray_size}" z="${ray_size}" />
-  </link>
-  <joint name="ray_joint" type="fixed">
-    <axis xyz="0 1 0" />
-    <origin xyz="${hull_loa/2 - 0.25} 0.4 ${hull_doa/2 + ray_size/2}" rpy="0 0 0"/>
-    <parent link="base_link"/>
-    <child link="ray_link"/>
-  </joint>
- <!-- GPS -->
-  <link name="gps_link">
-    <visual>
-      <geometry>
-        <box size="${gps_size} ${gps_size} ${gps_size}"/>
-      </geometry>
-      <material name="red" />
-    </visual>
-    <collision>
-      <geometry>
-        <box size="${gps_size} ${gps_size} ${gps_size}"/>
-      </geometry>
-    </collision>
-    <xacro:box_inertial mass="${gps_mass}" x="${gps_size}" y="${gps_size}" z="${gps_size}" />
-  </link>
-  <joint name="gps_joint" type="fixed">
-    <axis xyz="0 1 0" />
-    <origin xyz="0 0.4 ${hull_doa/2 + gps_size/2}" rpy="0 0 0"/>
-    <parent link="base_link"/>
-    <child link="gps_link"/>
-  </joint>
- <!-- IMU -->
-  <link name="imu_link">
-    <visual>
-      <geometry>
-        <box size="${imu_size} ${imu_size} ${imu_size}"/>
-      </geometry>
-      <material name="red" />
-    </visual>
-    <collision>
-      <geometry>
-        <box size="${imu_size} ${imu_size} ${imu_size}"/>
-      </geometry>
-    </collision>
-    <xacro:box_inertial mass="${imu_mass}" x="${imu_size}" y="${imu_size}" z="${imu_size}" />
-  </link>
-  <joint name="imu_joint" type="fixed">
-    <axis xyz="0 1 0" />
-    <origin xyz="0 0 ${hull_doa/2 + imu_size/2}" rpy="0 0 0"/>
-    <parent link="base_link"/>
-    <child link="imu_link"/>
-  </joint>
-   <!-- Magnetometer -->
-  <link name="mag_link">
-    <visual>
-      <geometry>
-        <box size="${mag_size} ${mag_size} ${mag_size}"/>
-      </geometry>
-      <material name="red" />
-    </visual>
-    <collision>
-      <geometry>
-        <box size="${mag_size} ${mag_size} ${mag_size}"/>
-      </geometry>
-    </collision>
-    <xacro:box_inertial mass="${gps_mass}" x="${mag_size}" y="${mag_size}" z="${mag_size}" />
-  </link>
-  <joint name="mag_joint" type="fixed">
-    <axis xyz="0 1 0" />
-    <origin xyz="0 -0.4 ${hull_doa/2 + mag_size/2}" rpy="0 0 0"/>
-    <parent link="base_link"/>
-    <child link="mag_link"/>
-  </joint>
+<!--
+    Software License Agreement (BSD-3-Clause)
+    Copyright (c) 2020 Rhys Mainwaring
+    All rights reserved.
+    Redistribution and use in source and binary forms, with or without
+    modification, are permitted provided that the following conditions
+    are met:
+    1.  Redistributions of source code must retain the above copyright
+        notice, this list of conditions and the following disclaimer.
+    2.  Redistributions in binary form must reproduce the above
+        copyright notice, this list of conditions and the following
+        disclaimer in the documentation and/or other materials provided
+        with the distribution.
+    3.  Neither the name of the copyright holder nor the names of its
+        contributors may be used to endorse or promote products derived
+        from this software without specific prior written permission.
+    THIS SOFTWARE IS PROVIDED BY THE COPYRIGHT HOLDERS AND CONTRIBUTORS
+    "AS IS" AND ANY EXPRESS OR IMPLIED WARRANTIES, INCLUDING, BUT NOT
+    LIMITED TO, THE IMPLIED WARRANTIES OF MERCHANTABILITY AND FITNESS
+    FOR A PARTICULAR PURPOSE ARE DISCLAIMED. IN NO EVENT SHALL THE
+    COPYRIGHT HOLDER OR CONTRIBUTORS BE LIABLE FOR ANY DIRECT, INDIRECT,
+    INCIDENTAL, SPECIAL, EXEMPLARY, OR CONSEQUENTIAL DAMAGES (INCLUDING,
+    BUT NOT LIMITED TO, PROCUREMENT OF SUBSTITUTE GOODS OR SERVICES;
+    LOSS OF USE, DATA, OR PROFITS; OR BUSINESS INTERRUPTION) HOWEVER
+    CAUSED AND ON ANY THEORY OF LIABILITY, WHETHER IN CONTRACT, STRICT
+    LIABILITY, OR TORT (INCLUDING NEGLIGENCE OR OTHERWISE) ARISING IN
+    ANY WAY OUT OF THE USE OF THIS SOFTWARE, EVEN IF ADVISED OF THE
+    POSSIBILITY OF SUCH DAMAGE.
+-->
+<!-- Robot description for a RS750 yacht
+ -->
+<robot name="rs750" xmlns:xacro="http://www.ros.org/wiki/xacro">
+    <xacro:include filename="$(find rs750_description)/urdf/rs750_materials.xacro"/>
+    <xacro:include filename="$(find rs750_description)/urdf/rs750_inertials.xacro"/>
+    <!-- Constants for robot dimensions -->
+    <xacro:property name="hull_mass" value="20000.0" />
+    <xacro:property name="hull_loa" value="10.0" />
+    <xacro:property name="hull_woa" value="4.0" />
+    <xacro:property name="hull_doa" value="2.0" />
+    <xacro:property name="cam_mass" value="0.1" />
+    <xacro:property name="cam_size" value="0.1" />
+    <xacro:property name="ray_mass" value="0.1" />
+    <xacro:property name="ray_size" value="0.1" />
+    <xacro:property name="imu_mass" value="0.1" />
+    <xacro:property name="imu_size" value="0.1" />
+    <xacro:property name="gps_mass" value="0.1" />
+    <xacro:property name="gps_size" value="0.1" />
+    <xacro:property name="mag_mass" value="0.1" />
+    <xacro:property name="mag_size" value="0.1" />
+    <!-- Base link (main hull) -->
+    <link name="base_link">
+        <visual>
+            <geometry>
+                <box size="${hull_loa} ${hull_woa} ${hull_doa}"/>
+            </geometry>
+            <material name="orange" />
+        </visual>
+        <collision>
+            <geometry>
+                <box size="${hull_loa} ${hull_woa} ${hull_doa}"/>
+            </geometry>
+        </collision>
+        <xacro:box_inertial mass="${hull_mass}" x="${hull_loa}" y="${hull_loa}" z="${hull_doa}" />
+    </link>
+    <!-- Camera -->
+    <link name="cam_link">
+        <visual>
+            <geometry>
+                <box size="${cam_size} ${cam_size} ${cam_size}"/>
+            </geometry>
+            <material name="red" />
+        </visual>
+        <collision>
+            <geometry>
+                <box size="${cam_size} ${cam_size} ${cam_size}"/>
+            </geometry>
+        </collision>
+        <xacro:box_inertial mass="${cam_mass}" x="${cam_size}" y="${cam_size}" z="${cam_size}" />
+    </link>
+    <joint name="cam_joint" type="fixed">
+        <axis xyz="0 1 0" />
+        <origin xyz="${hull_loa/2 - 0.25} 0 ${hull_doa/2 + cam_size/2}" rpy="0 0 0"/>
+        <parent link="base_link"/>
+        <child link="cam_link"/>
+    </joint>
+    <!-- Ray -->
+    <link name="ray_link">
+        <visual>
+            <geometry>
+              <box size="${ray_size} ${ray_size} ${ray_size}"/>
+            </geometry>
+            <material name="red" />
+        </visual>
+        <collision>
+            <geometry>
+                <box size="${ray_size} ${ray_size} ${ray_size}"/>
+            </geometry>
+        </collision>
+        <xacro:box_inertial mass="${ray_mass}" x="${ray_size}" y="${ray_size}" z="${ray_size}" />
+    </link>
+    <joint name="ray_joint" type="fixed">
+        <axis xyz="0 1 0" />
+        <origin xyz="${hull_loa/2 - 0.25} 0.4 ${hull_doa/2 + ray_size/2}" rpy="0 0 0"/>
+        <parent link="base_link"/>
+        <child link="ray_link"/>
+    </joint>
+    <!-- GPS -->
+    <link name="gps_link">
+        <visual>
+            <geometry>
+                <box size="${gps_size} ${gps_size} ${gps_size}"/>
+            </geometry>
+            <material name="red" />
+        </visual>
+        <collision>
+            <geometry>
+                <box size="${gps_size} ${gps_size} ${gps_size}"/>
+            </geometry>
+        </collision>
+        <xacro:box_inertial mass="${gps_mass}" x="${gps_size}" y="${gps_size}" z="${gps_size}" />
+    </link>
+    <joint name="gps_joint" type="fixed">
+        <axis xyz="0 1 0" />
+        <origin xyz="0 0.4 ${hull_doa/2 + gps_size/2}" rpy="0 0 0"/>
+        <parent link="base_link"/>
+        <child link="gps_link"/>
+    </joint>
+    <!-- IMU -->
+    <link name="imu_link">
+        <visual>
+            <geometry>
+                <box size="${imu_size} ${imu_size} ${imu_size}"/>
+            </geometry>
+            <material name="red" />
+        </visual>
+        <collision>
+            <geometry>
+                <box size="${imu_size} ${imu_size} ${imu_size}"/>
+            </geometry>
+        </collision>
+        <xacro:box_inertial mass="${imu_mass}" x="${imu_size}" y="${imu_size}" z="${imu_size}" />
+    </link>
+    <joint name="imu_joint" type="fixed">
+        <axis xyz="0 1 0" />
+        <origin xyz="0 0 ${hull_doa/2 + imu_size/2}" rpy="0 0 0"/>
+        <parent link="base_link"/>
+        <child link="imu_link"/>
+    </joint>
+    <!-- Magnetometer -->
+    <link name="mag_link">
+        <visual>
+            <geometry>
+                <box size="${mag_size} ${mag_size} ${mag_size}"/>
+            </geometry>
+            <material name="red" />
+        </visual>
+        <collision>
+            <geometry>
+                <box size="${mag_size} ${mag_size} ${mag_size}"/>
+            </geometry>
+        </collision>
+        <xacro:box_inertial mass="${gps_mass}" x="${mag_size}" y="${mag_size}" z="${mag_size}" />
+    </link>
+    <joint name="mag_joint" type="fixed">
+        <axis xyz="0 1 0" />
+        <origin xyz="0 -0.4 ${hull_doa/2 + mag_size/2}" rpy="0 0 0"/>
+        <parent link="base_link"/>
+        <child link="mag_link"/>
+    </joint>
 </robot>

File: rs750_description/urdf/rs750_materials.xacro (robot description, xacro)
@@ -1,18 +1,61 @@
 <?xml version="1.0" ?>
-<robot>
-  <material name="black">
-    <color rgba="0.0 0.0 0.0 1.0"/>
-  </material>
-  <material name="red">
-    <color rgba="0.8 0.0 0.0 1.0"/>
-  </material>
-  <material name="green">
-    <color rgba="0.0 0.8 0.0 1.0"/>
-  </material>
-  <material name="blue">
-    <color rgba="0.0 0.0 0.8 1.0"/>
-  </material>
-  <material name="orange">
-    <color rgba="${255/255} ${108/255} ${10/255} 1.0"/>
-  </material>
+<!--
+    Software License Agreement (BSD-3-Clause)
+    Copyright (c) 2020 Rhys Mainwaring
+    All rights reserved.
+    Redistribution and use in source and binary forms, with or without
+    modification, are permitted provided that the following conditions
+    are met:
+    1.  Redistributions of source code must retain the above copyright
+        notice, this list of conditions and the following disclaimer.
+    2.  Redistributions in binary form must reproduce the above
+        copyright notice, this list of conditions and the following
+        disclaimer in the documentation and/or other materials provided
+        with the distribution.
+    3.  Neither the name of the copyright holder nor the names of its
+        contributors may be used to endorse or promote products derived
+        from this software without specific prior written permission.
+    THIS SOFTWARE IS PROVIDED BY THE COPYRIGHT HOLDERS AND CONTRIBUTORS
+    "AS IS" AND ANY EXPRESS OR IMPLIED WARRANTIES, INCLUDING, BUT NOT
+    LIMITED TO, THE IMPLIED WARRANTIES OF MERCHANTABILITY AND FITNESS
+    FOR A PARTICULAR PURPOSE ARE DISCLAIMED. IN NO EVENT SHALL THE
+    COPYRIGHT HOLDER OR CONTRIBUTORS BE LIABLE FOR ANY DIRECT, INDIRECT,
+    INCIDENTAL, SPECIAL, EXEMPLARY, OR CONSEQUENTIAL DAMAGES (INCLUDING,
+    BUT NOT LIMITED TO, PROCUREMENT OF SUBSTITUTE GOODS OR SERVICES;
+    LOSS OF USE, DATA, OR PROFITS; OR BUSINESS INTERRUPTION) HOWEVER
+    CAUSED AND ON ANY THEORY OF LIABILITY, WHETHER IN CONTRACT, STRICT
+    LIABILITY, OR TORT (INCLUDING NEGLIGENCE OR OTHERWISE) ARISING IN
+    ANY WAY OUT OF THE USE OF THIS SOFTWARE, EVEN IF ADVISED OF THE
+    POSSIBILITY OF SUCH DAMAGE.
+-->
+<!--  xacro macros for robot materials.
+ -->
+<robot name="rs750_materials" xmlns:xacro="http://ros.org/wiki/xacro">
+   <material name="red">
+        <color rgba="0.8 0 0 1"/>
+    </material>
+    <material name="green">
+        <color rgba="0 0.8 0 1"/>
+    </material>
+    <material name="blue">
+        <color rgba="0 0 0.8 1"/>
+    </material>
+    <material name="orange">
+        <color rgba="0.8 0.25 0 1"/>
+    </material>
+    <material name="black">
+        <color rgba="0 0 0 1"/>
+    </material>
+    <material name="dark_gray">
+        <color rgba="0.5 0.5 0.5 1"/>
+    </material>
+    <material name="gray">
+        <color rgba="0.753 0.753 0.753 1"/>
+    </material>
+    <material name="silver">
+        <color rgba="0.88 0.88 0.88 1"/>
+    </material>
+    <material name="white">
+        <color rgba="1 1 1 1"/>
+    </material>
 </robot>

Commit message: Update robot description. Add hull and deck elements.
1. Add hull and deck visual and collision elements.
2. Update dimensions from RS 750 specifications (mass is approx)

File: rs750_description/urdf/rs750.urdf.xacro (robot description, xacro)
@@ -35,8 +35,8 @@
     <xacro:include filename="$(find rs750_description)/urdf/rs750_inertials.xacro"/>
     <!-- Constants for robot dimensions -->
-    <xacro:property name="hull_mass" value="20000.0" />
-    <xacro:property name="hull_loa" value="10.0" />
-    <xacro:property name="hull_woa" value="4.0" />
-    <xacro:property name="hull_doa" value="2.0" />
+    <xacro:property name="hull_mass" value="1.0" />
+    <xacro:property name="hull_loa" value="0.770" />
+    <xacro:property name="hull_woa" value="0.150" />
+    <xacro:property name="hull_doa" value="0.080" />
     <xacro:property name="cam_mass" value="0.1" />
     <xacro:property name="cam_size" value="0.1" />
@@ -49,21 +49,68 @@
     <xacro:property name="mag_mass" value="0.1" />
     <xacro:property name="mag_size" value="0.1" />
-    <!-- Base link (main hull) -->
+    <!-- The base link - the reference link for the entire model -->
     <link name="base_link">
         <visual>
-            <geometry>
-                <box size="${hull_loa} ${hull_woa} ${hull_doa}"/>
+            <origin rpy="0 0 0" xyz="0 0 0" />
+            <geometry>
+                <box size="0.01 0.01 0.01"/>
             </geometry>
             <material name="orange" />
         </visual>
         <collision>
-            <geometry>
-                <box size="${hull_loa} ${hull_woa} ${hull_doa}"/>
-            </geometry>
-        </collision>
-        <xacro:box_inertial mass="${hull_mass}" x="${hull_loa}" y="${hull_loa}" z="${hull_doa}" />
-    </link>
+            <origin rpy="0 0 0" xyz="0 0 0" />
+            <geometry>
+                <box size="0.01 0.01 0.01"/>
+            </geometry>
+        </collision>
+        <xacro:solid_cuboid_inertial
+            rpy="0 0 0" xyz="0 0 0"
+            mass="0.01"
+            x="0.01" y="0.01" z="0.01" />
+    </link>
+    <gazebo reference="base_link">
+        <material>Gazebo/Orange</material>
+    </gazebo>
+    <!-- Hull  -->
+    <link name="hull_link">
+        <visual name="hull_visual">
+            <origin rpy="0 0 0" xyz="0 0 0" />
+            <geometry>
+                <mesh filename="package://rs750_description/meshes/rs750_hull.stl" />
+            </geometry>
+            <material name="red" />
+        </visual>
+        <visual name="deck_visual">
+            <origin rpy="0 0 0" xyz="0 0 0" />
+            <geometry>
+                <mesh filename="package://rs750_description/meshes/rs750_deck.stl" />
+            </geometry>
+            <material name="dark_gray" />
+        </visual>
+        <collision>
+            <origin rpy="0 0 0" xyz="0 0 0" />
+            <geometry>
+                <mesh filename="package://rs750_description/meshes/rs750_hull_collision.stl" />
+            </geometry>
+        </collision>
+        <xacro:solid_cuboid_inertial
+            rpy="0 0 0" xyz="0 0 0"
+            mass="${hull_mass}"
+            x="${hull_loa}" y="${hull_woa}" z="${hull_doa}" />
+    </link>
+    <gazebo reference="hull_link">
+        <material>Gazebo/DarkGray</material>
+    </gazebo>
+    <joint name="hull_joint" type="fixed">
+        <origin rpy="0 0 0" xyz="0 0 0"/>
+        <parent link="base_link" />
+        <child link="hull_link" />
+    </joint>
+    <gazebo reference="hull_joint">
+        <!-- <disableFixedJointLumping>true</disableFixedJointLumping>  -->
+        <!-- <preserveFixedJoint>true</preserveFixedJoint> -->
+    </gazebo>
     <!-- Camera -->
-    <link name="cam_link">
+    <!-- <link name="cam_link">
         <visual>
             <geometry>
@@ -77,5 +124,5 @@
             </geometry>
         </collision>
-        <xacro:box_inertial mass="${cam_mass}" x="${cam_size}" y="${cam_size}" z="${cam_size}" />
+        <xacro:solid_cuboid_inertial mass="${cam_mass}" x="${cam_size}" y="${cam_size}" z="${cam_size}" />
     </link>
     <joint name="cam_joint" type="fixed">
@@ -84,7 +131,7 @@
         <parent link="base_link"/>
         <child link="cam_link"/>
-    </joint>
+    </joint> -->
     <!-- Ray -->
-    <link name="ray_link">
+    <!-- <link name="ray_link">
         <visual>
             <geometry>
@@ -98,5 +145,5 @@
             </geometry>
         </collision>
-        <xacro:box_inertial mass="${ray_mass}" x="${ray_size}" y="${ray_size}" z="${ray_size}" />
+        <xacro:solid_cuboid_inertial mass="${ray_mass}" x="${ray_size}" y="${ray_size}" z="${ray_size}" />
     </link>
     <joint name="ray_joint" type="fixed">
@@ -105,7 +152,7 @@
         <parent link="base_link"/>
         <child link="ray_link"/>
-    </joint>
+    </joint> -->
     <!-- GPS -->
-    <link name="gps_link">
+    <!-- <link name="gps_link">
         <visual>
             <geometry>
@@ -119,5 +166,5 @@
             </geometry>
         </collision>
-        <xacro:box_inertial mass="${gps_mass}" x="${gps_size}" y="${gps_size}" z="${gps_size}" />
+        <xacro:solid_cuboid_inertial mass="${gps_mass}" x="${gps_size}" y="${gps_size}" z="${gps_size}" />
     </link>
     <joint name="gps_joint" type="fixed">
@@ -126,7 +173,7 @@
         <parent link="base_link"/>
         <child link="gps_link"/>
-    </joint>
+    </joint> -->
     <!-- IMU -->
-    <link name="imu_link">
+    <!-- <link name="imu_link">
         <visual>
             <geometry>
@@ -140,5 +187,5 @@
             </geometry>
         </collision>
-        <xacro:box_inertial mass="${imu_mass}" x="${imu_size}" y="${imu_size}" z="${imu_size}" />
+        <xacro:solid_cuboid_inertial mass="${imu_mass}" x="${imu_size}" y="${imu_size}" z="${imu_size}" />
     </link>
     <joint name="imu_joint" type="fixed">
@@ -147,7 +194,7 @@
         <parent link="base_link"/>
         <child link="imu_link"/>
-    </joint>
+    </joint> -->
     <!-- Magnetometer -->
-    <link name="mag_link">
+    <!-- <link name="mag_link">
         <visual>
             <geometry>
@@ -161,5 +208,5 @@
             </geometry>
         </collision>
-        <xacro:box_inertial mass="${gps_mass}" x="${mag_size}" y="${mag_size}" z="${mag_size}" />
+        <xacro:solid_cuboid_inertial mass="${gps_mass}" x="${mag_size}" y="${mag_size}" z="${mag_size}" />
     </link>
     <joint name="mag_joint" type="fixed">
@@ -168,4 +215,4 @@
         <parent link="base_link"/>
         <child link="mag_link"/>
-    </joint>
+    </joint> -->
 </robot>
