Commit message: Add rudder and keel.
1. Add elements for rudder and keel
2. Add revolute joint for rudder

File: rs750_description/urdf/rs750.urdf.xacro (robot description, xacro)
@@ -30,4 +30,9 @@
 -->
 <!-- Robot description for a RS750 yacht
+    Conventions
+    ROS REP 105 Coordinate Frames for Mobile Platforms
+    length      x-axis dimension
+    width       y-axis dimension
+    depth       z-axis dimension
  -->
 <robot name="rs750" xmlns:xacro="http://www.ros.org/wiki/xacro">
@@ -35,8 +40,21 @@
     <xacro:include filename="$(find rs750_description)/urdf/rs750_inertials.xacro"/>
     <!-- Constants for robot dimensions -->
-    <xacro:property name="hull_mass" value="1.0" />
-    <xacro:property name="hull_loa" value="0.770" />
-    <xacro:property name="hull_woa" value="0.150" />
-    <xacro:property name="hull_doa" value="0.080" />
+    <xacro:property name="scale" value="3.2" />
+    <xacro:property name="volume_scale" value="${scale * scale * scale}" />
+    <xacro:property name="hull_mass" value="${1.0 * volume_scale}" />
+    <xacro:property name="hull_length" value="${0.770 * scale}" />
+    <xacro:property name="hull_width" value="${0.150 * scale}" />
+    <xacro:property name="hull_depth" value="${0.080 * scale}" />
+    <xacro:property name="keel_fin_mass" value="${0.250 * volume_scale}" />
+    <xacro:property name="keel_fin_length" value="${0.040 * scale}" />
+    <xacro:property name="keel_fin_width" value="${0.006 * scale}" />
+    <xacro:property name="keel_fin_depth" value="${0.270 * scale}" />
+    <xacro:property name="keel_bulb_mass" value="${1.30 * volume_scale}" />
+    <xacro:property name="keel_bulb_length" value="${0.215 * scale}" />
+    <xacro:property name="keel_bulb_radius" value="${0.015 * scale}" />
+    <xacro:property name="rudder_mass" value="${0.100 * volume_scale}" />
+    <xacro:property name="rudder_length" value="${0.040 * scale}" />
+    <xacro:property name="rudder_width" value="${0.006 * scale}" />
+    <xacro:property name="rudder_depth" value="${0.160 * scale}" />
     <xacro:property name="cam_mass" value="0.1" />
     <xacro:property name="cam_size" value="0.1" />
@@ -64,8 +82,15 @@
             </geometry>
         </collision>
+        <!-- Remove inertial in base_link:
+            [ WARN ] The root link base_link has an inertia specified in the URDF,
+            but KDL does not support a root link with an inertia.
+            As a workaround, you can add an extra dummy link to your URDF.
+        -->
+        <!--
         <xacro:solid_cuboid_inertial
             rpy="0 0 0" xyz="0 0 0"
             mass="0.01"
             x="0.01" y="0.01" z="0.01" />
+        -->
     </link>
     <gazebo reference="base_link">
@@ -88,8 +113,8 @@
             <material name="dark_gray" />
         </visual>
-        <collision>
-            <origin rpy="0 0 0" xyz="0 0 0" />
-            <geometry>
-                <mesh filename="package://rs750_description/meshes/rs750_hull_collision.stl" />
+        <collision name="hull_collision">
+            <origin rpy="0 0 0" xyz="0 0 0" />
+            <geometry>
+                <mesh filename="package://rs750_description/meshes/rs750_hull_collision_3.stl" />
             </geometry>
         </collision>
@@ -97,8 +122,8 @@
             rpy="0 0 0" xyz="0 0 0"
             mass="${hull_mass}"
-            x="${hull_loa}" y="${hull_woa}" z="${hull_doa}" />
+            x="${hull_length}" y="${hull_width}" z="${hull_depth}" />
     </link>
     <gazebo reference="hull_link">
-        <material>Gazebo/DarkGray</material>
+        <material>Gazebo/Red</material>
     </gazebo>
     <joint name="hull_joint" type="fixed">
@@ -108,6 +133,101 @@
     </joint>
     <gazebo reference="hull_joint">
-        <!-- <disableFixedJointLumping>true</disableFixedJointLumping>  -->
-        <!-- <preserveFixedJoint>true</preserveFixedJoint> -->
+    </gazebo>
+    <!-- Keel fin -->
+    <link name="keel_fin_link">
+        <visual name="keel_fin_visual">
+            <origin rpy="0 0 0" xyz="0 0 0" />
+            <geometry>
+                <mesh filename="package://rs750_description/meshes/rs750_keel_fin.stl" />
+            </geometry>
+            <material name="yellow" />
+        </visual>
+        <collision name="keel_fin_collision">
+            <origin rpy="0 0 0" xyz="0 0 0" />
+            <geometry>
+                <mesh filename="package://rs750_description/meshes/rs750_keel_fin_collision_2.stl" />
+            </geometry>
+        </collision>
+        <xacro:solid_cuboid_inertial
+            rpy="0 0 0" xyz="0 0 0"
+            mass="${keel_fin_mass}"
+            x="${keel_fin_length}" y="${keel_fin_width}" z="${keel_fin_depth}" />
+    </link>
+    <gazebo reference="keel_fin_link">
+        <material>Gazebo/Yellow</material>
+    </gazebo>
+    <joint name="keel_fin_joint" type="fixed">
+        <origin rpy="0 0 0" xyz="-0.16255 0.0 -0.54053"/>
+        <parent link="base_link" />
+        <child link="keel_fin_link" />
+    </joint>
+    <gazebo reference="keel_fin_joint">
+    </gazebo>
+    <!-- Keel bulb -->
+    <link name="keel_bulb_link">
+        <visual name="keel_bulb_visual">
+            <origin rpy="0 0 0" xyz="0 0 0" />
+            <geometry>
+                <mesh filename="package://rs750_description/meshes/rs750_keel_bulb.stl" />
+            </geometry>
+            <material name="yellow" />
+        </visual>
+        <collision name="keel_bulb_collision">
+            <origin rpy="0 ${math_pi_over_2} 0" xyz="0 0 0" />
+            <geometry>
+                <cylinder length="${keel_bulb_length}" radius="${keel_bulb_radius}" />
+            </geometry>
+        </collision>
+        <xacro:solid_cylinder_inertial
+            rpy="0 ${math_pi_over_2} 0" xyz="0 0 0"
+            mass="${keel_bulb_mass}"
+            radius="${keel_bulb_radius}" length="${keel_bulb_length}" />
+    </link>
+    <gazebo reference="keel_bulb_link">
+        <material>Gazebo/Yellow</material>
+    </gazebo>
+    <joint name="keel_bulb_joint" type="fixed">
+        <origin rpy="0 0 0" xyz="-0.26638 0.0 -1.08674"/>
+        <parent link="base_link" />
+        <child link="keel_bulb_link" />
+    </joint>
+    <gazebo reference="keel_bulb_joint">
+    </gazebo>
+    <!-- Rudder -->
+    <link name="rudder_link">
+        <visual name="rudder_visual">
+            <origin rpy="0 0 0" xyz="0 0 0" />
+            <geometry>
+                <mesh filename="package://rs750_description/meshes/rs750_rudder.stl" />
+            </geometry>
+            <material name="yellow" />
+        </visual>
+        <collision name="rudder_collision">
+            <origin rpy="0 0 0" xyz="0 0 0" />
+            <geometry>
+                <mesh filename="package://rs750_description/meshes/rs750_rudder_collision_3.stl" />
+            </geometry>
+        </collision>
+        <xacro:solid_cuboid_inertial
+            rpy="0 0 0" xyz="0 0 0"
+            mass="${rudder_mass}"
+            x="${rudder_length}" y="${rudder_width}" z="${rudder_depth}" />
+    </link>
+    <gazebo reference="rudder_link">
+        <material>Gazebo/Yellow</material>
+    </gazebo>
+    <joint name="rudder_joint" type="revolute">
+        <origin rpy="0 0 0" xyz="-1.2436 0.0 -0.0487"/>
+        <axis xyz="0 0 1" />
+        <limit
+            lower="${-math_pi_over_2}"
+            upper="${-math_pi_over_2}"
+            effort="10000"
+            velocity="10000"
+        />
+        <parent link="base_link" />
+        <child link="rudder_link" />
+    </joint>
+    <gazebo reference="rudder_joint">
     </gazebo>
     <!-- Camera -->
@@ -128,5 +248,5 @@
     <joint name="cam_joint" type="fixed">
         <axis xyz="0 1 0" />
-        <origin xyz="${hull_loa/2 - 0.25} 0 ${hull_doa/2 + cam_size/2}" rpy="0 0 0"/>
+        <origin xyz="${hull_length/2 - 0.25} 0 ${hull_depth/2 + cam_size/2}" rpy="0 0 0"/>
         <parent link="base_link"/>
         <child link="cam_link"/>
@@ -149,5 +269,5 @@
     <joint name="ray_joint" type="fixed">
         <axis xyz="0 1 0" />
-        <origin xyz="${hull_loa/2 - 0.25} 0.4 ${hull_doa/2 + ray_size/2}" rpy="0 0 0"/>
+        <origin xyz="${hull_length/2 - 0.25} 0.4 ${hull_depth/2 + ray_size/2}" rpy="0 0 0"/>
         <parent link="base_link"/>
         <child link="ray_link"/>
@@ -170,5 +290,5 @@
     <joint name="gps_joint" type="fixed">
         <axis xyz="0 1 0" />
-        <origin xyz="0 0.4 ${hull_doa/2 + gps_size/2}" rpy="0 0 0"/>
+        <origin xyz="0 0.4 ${hull_depth/2 + gps_size/2}" rpy="0 0 0"/>
         <parent link="base_link"/>
         <child link="gps_link"/>
@@ -191,5 +311,5 @@
     <joint name="imu_joint" type="fixed">
         <axis xyz="0 1 0" />
-        <origin xyz="0 0 ${hull_doa/2 + imu_size/2}" rpy="0 0 0"/>
+        <origin xyz="0 0 ${hull_depth/2 + imu_size/2}" rpy="0 0 0"/>
         <parent link="base_link"/>
         <child link="imu_link"/>
@@ -212,5 +332,5 @@
     <joint name="mag_joint" type="fixed">
         <axis xyz="0 1 0" />
-        <origin xyz="0 -0.4 ${hull_doa/2 + mag_size/2}" rpy="0 0 0"/>
+        <origin xyz="0 -0.4 ${hull_depth/2 + mag_size/2}" rpy="0 0 0"/>
         <parent link="base_link"/>
         <child link="mag_link"/>

File: rs750_description/urdf/rs750_materials.xacro (robot description, xacro)
@@ -44,4 +44,7 @@
         <color rgba="0.8 0.25 0 1"/>
     </material>
+    <material name="yellow">
+        <color rgba="0.8 0.8 0 1"/>
+    </material>
     <material name="black">
         <color rgba="0 0 0 1"/>

Commit message: Add launch files for Gazebo simulation.
1. Include the gazebo elements for the wave field and hydrodynamics plugin.
2. Remove name attributes for visuals and collisions (they prevent the gazebo materials from being used)

File: rs750_description/urdf/rs750.urdf.xacro (robot description, xacro)
@@ -39,4 +39,5 @@
     <xacro:include filename="$(find rs750_description)/urdf/rs750_materials.xacro"/>
     <xacro:include filename="$(find rs750_description)/urdf/rs750_inertials.xacro"/>
+    <xacro:include filename="$(find rs750_description)/urdf/rs750.gazebo"/>
     <!-- Constants for robot dimensions -->
     <xacro:property name="scale" value="3.2" />
@@ -99,5 +100,5 @@
     <!-- Hull  -->
     <link name="hull_link">
-        <visual name="hull_visual">
+        <visual>
             <origin rpy="0 0 0" xyz="0 0 0" />
             <geometry>
@@ -106,5 +107,5 @@
             <material name="red" />
         </visual>
-        <visual name="deck_visual">
+        <visual>
             <origin rpy="0 0 0" xyz="0 0 0" />
             <geometry>
@@ -136,5 +137,5 @@
     <!-- Keel fin -->
     <link name="keel_fin_link">
-        <visual name="keel_fin_visual">
+        <visual>
             <origin rpy="0 0 0" xyz="0 0 0" />
             <geometry>
@@ -143,5 +144,5 @@
             <material name="yellow" />
         </visual>
-        <collision name="keel_fin_collision">
+        <collision>
             <origin rpy="0 0 0" xyz="0 0 0" />
             <geometry>
@@ -166,5 +167,5 @@
     <!-- Keel bulb -->
     <link name="keel_bulb_link">
-        <visual name="keel_bulb_visual">
+        <visual>
             <origin rpy="0 0 0" xyz="0 0 0" />
             <geometry>
@@ -173,5 +174,5 @@
             <material name="yellow" />
         </visual>
-        <collision name="keel_bulb_collision">
+        <collision>
             <origin rpy="0 ${math_pi_over_2} 0" xyz="0 0 0" />
             <geometry>
@@ -196,5 +197,5 @@
     <!-- Rudder -->
     <link name="rudder_link">
-        <visual name="rudder_visual">
+        <visual>
             <origin rpy="0 0 0" xyz="0 0 0" />
             <geometry>
@@ -203,5 +204,5 @@
             <material name="yellow" />
         </visual>
-        <collision name="rudder_collision">
+        <collision>
             <origin rpy="0 0 0" xyz="0 0 0" />
             <geometry>

File: rs750_description/urdf/rs750_inertials.xacro (robot description, xacro)
@@ -35,5 +35,5 @@
     - null (a placeholder inertial for logical link elements)
  -->
-<robot name="rs750_inertials" xmlns:xacro="http://ros.org/wiki/xacro">
+<robot xmlns:xacro="http://www.ros.org/wiki/xacro">
     <!-- Math constants -->
     <xacro:property name="math_pi"        value="3.141592653589793" />

File: rs750_description/urdf/rs750_materials.xacro (robot description, xacro)
@@ -31,5 +31,5 @@
 <!--  xacro macros for robot materials.
  -->
-<robot name="rs750_materials" xmlns:xacro="http://ros.org/wiki/xacro">
+<robot xmlns:xacro="http://www.ros.org/wiki/xacro">
    <material name="red">
         <color rgba="0.8 0 0 1"/>

Commit message: Add rig elements to robot model.
1. Add fore and main sails to robot model.
2. Update rviz launch file to use gui version of the joint state publisher when option is set.
3. Update rviz config file.

File: rs750_description/urdf/rs750.urdf.xacro (robot description, xacro)
@@ -58,4 +58,14 @@
     <xacro:property name="rudder_width" value="${0.006 * scale}" />
     <xacro:property name="rudder_depth" value="${0.160 * scale}" />
+    <!-- Rough estimates for intertial -->
+    <xacro:property name="main_sail_mass" value="${0.100 * volume_scale}" />
+    <xacro:property name="main_sail_length" value="${0.200 * scale}" />
+    <xacro:property name="main_sail_width" value="${0.006 * scale}" />
+    <xacro:property name="main_sail_depth" value="${0.900 * scale}" />
+    <!-- Rough estimates for intertial -->
+    <xacro:property name="fore_sail_mass" value="${0.0500 * volume_scale}" />
+    <xacro:property name="fore_sail_length" value="${0.100 * scale}" />
+    <xacro:property name="fore_sail_width" value="${0.006 * scale}" />
+    <xacro:property name="fore_sail_depth" value="${0.700 * scale}" />
     <xacro:property name="cam_mass" value="0.1" />
     <xacro:property name="cam_size" value="0.1" />
@@ -232,4 +242,98 @@
     <gazebo reference="rudder_joint">
     </gazebo>
+    <!-- Mast -->
+    <link name="mast_link">
+        <visual>
+            <origin rpy="0 0 0" xyz="0 0 0" />
+            <geometry>
+                <mesh filename="package://rs750_description/meshes/rs750_mast.stl" />
+            </geometry>
+            <material name="black" />
+        </visual>
+    </link>
+    <gazebo reference="mast_link">
+        <material>Gazebo/Black</material>
+    </gazebo>
+    <joint name="mast_joint" type="fixed">
+        <origin rpy="0 0 0" xyz="0 0 2.09"/>
+        <parent link="base_link" />
+        <child link="mast_link" />
+    </joint>
+    <gazebo reference="mast_joint">
+    </gazebo>
+    <!-- Main sail -->
+    <link name="main_sail_link">
+        <visual>
+            <origin rpy="0 0 0" xyz="0 0 0" />
+            <geometry>
+                <mesh filename="package://rs750_description/meshes/rs750_main_sail.stl" />
+            </geometry>
+            <material name="gray" />
+        </visual>
+        <collision>
+            <origin rpy="0 0 0" xyz="0 0 0" />
+            <geometry>
+                <mesh filename="package://rs750_description/meshes/rs750_main_sail.stl" />
+            </geometry>
+        </collision>
+        <xacro:solid_cuboid_inertial
+            rpy="0 0 0" xyz="0 0 0"
+            mass="${main_sail_mass}"
+            x="${main_sail_length}" y="${main_sail_width}" z="${main_sail_depth}" />
+    </link>
+    <gazebo reference="main_sail_link">
+        <material>Gazebo/Gray</material>
+    </gazebo>
+    <joint name="main_sail_joint" type="revolute">
+        <origin rpy="0 0 0" xyz="-0.02625 0 0.291875"/>
+        <axis xyz="0 0 1" />
+        <limit
+            lower="${-math_pi_over_2}"
+            upper="${math_pi_over_2}"
+            effort="1000"
+            velocity="1000"
+        />
+        <parent link="base_link" />
+        <child link="main_sail_link" />
+    </joint>
+    <gazebo reference="main_sail_joint">
+    </gazebo>
+    <!-- Fore sail -->
+    <link name="fore_sail_link">
+        <visual>
+            <origin rpy="0 0 0" xyz="0 0 0" />
+            <geometry>
+                <mesh filename="package://rs750_description/meshes/rs750_fore_sail.stl" />
+            </geometry>
+            <material name="gray" />
+        </visual>
+        <collision>
+            <origin rpy="0 0 0" xyz="0 0 0" />
+            <geometry>
+                <mesh filename="package://rs750_description/meshes/rs750_fore_sail.stl" />
+            </geometry>
+        </collision>
+        <xacro:solid_cuboid_inertial
+            rpy="0 0 0" xyz="0 0 0"
+            mass="${fore_sail_mass}"
+            x="${fore_sail_length}" y="${fore_sail_width}" z="${fore_sail_depth}" />
+    </link>
+    <gazebo reference="fore_sail_link">
+        <material>Gazebo/Gray</material>
+    </gazebo>
+    <joint name="fore_sail_joint" type="revolute">
+        <origin rpy="0 0 0" xyz="1.03125 0 0.235625"/>
+        <axis xyz="-0.271652766 0 0.962395332" />
+        <limit
+            lower="${-math_pi_over_2}"
+            upper="${math_pi_over_2}"
+            effort="1000"
+            velocity="1000"
+        />
+        <parent link="base_link" />
+        <child link="fore_sail_link" />
+    </joint>
+    <gazebo reference="fore_sail_joint">
+    </gazebo>
     <!-- Camera -->
     <!-- <link name="cam_link">
