Commit message: Update robot description
1. Add urdf and gazebo sensor elements for imu and anemometer sensors.
2. Add lift/drag plugins for foils and sails

File: rs750_description/urdf/rs750.urdf.xacro (robot description, xacro)
@@ -39,4 +39,6 @@
     <xacro:include filename="$(find rs750_description)/urdf/rs750_materials.xacro"/>
     <xacro:include filename="$(find rs750_description)/urdf/rs750_inertials.xacro"/>
+    <xacro:include filename="$(find rs750_description)/urdf/rs750_imu.xacro"/>
+    <xacro:include filename="$(find rs750_description)/urdf/rs750_anemometer.xacro"/>
     <xacro:include filename="$(find rs750_description)/urdf/rs750.gazebo"/>
     <!-- Constants for robot dimensions -->
@@ -68,14 +70,4 @@
     <xacro:property name="fore_sail_width" value="${0.006 * scale}" />
     <xacro:property name="fore_sail_depth" value="${0.700 * scale}" />
-    <xacro:property name="cam_mass" value="0.1" />
-    <xacro:property name="cam_size" value="0.1" />
-    <xacro:property name="ray_mass" value="0.1" />
-    <xacro:property name="ray_size" value="0.1" />
-    <xacro:property name="imu_mass" value="0.1" />
-    <xacro:property name="imu_size" value="0.1" />
-    <xacro:property name="gps_mass" value="0.1" />
-    <xacro:property name="gps_size" value="0.1" />
-    <xacro:property name="mag_mass" value="0.1" />
-    <xacro:property name="mag_size" value="0.1" />
     <!-- The base link - the reference link for the entire model -->
     <link name="base_link">
@@ -117,11 +109,4 @@
             <material name="red" />
         </visual>
-        <visual>
-            <origin rpy="0 0 0" xyz="0 0 0" />
-            <geometry>
-                <mesh filename="package://rs750_description/meshes/rs750_deck.stl" />
-            </geometry>
-            <material name="dark_gray" />
-        </visual>
         <collision name="hull_collision">
             <origin rpy="0 0 0" xyz="0 0 0" />
@@ -145,4 +130,24 @@
     <gazebo reference="hull_joint">
     </gazebo>
+    <!-- Deck  (visual only) -->
+    <link name="deck_link">
+        <visual>
+            <origin rpy="0 0 0" xyz="0 0 0" />
+            <geometry>
+                <mesh filename="package://rs750_description/meshes/rs750_deck.stl" />
+            </geometry>
+            <material name="dark_gray" />
+        </visual>
+    </link>
+    <gazebo reference="deck_link">
+        <material>Gazebo/Gray</material>
+    </gazebo>
+    <joint name="deck_joint" type="fixed">
+        <origin rpy="0 0 0" xyz="0 0 0"/>
+        <parent link="base_link" />
+        <child link="deck_link" />
+    </joint>
+    <gazebo reference="deck_joint">
+    </gazebo>
     <!-- Keel fin -->
     <link name="keel_fin_link">
@@ -173,5 +178,8 @@
         <child link="keel_fin_link" />
     </joint>
+    <!-- Preserve fixed joint as the keel_fin_link has an associated plugin -->
     <gazebo reference="keel_fin_joint">
+        <disableFixedJointLumping>true</disableFixedJointLumping>
+        <preserveFixedJoint>true</preserveFixedJoint>
     </gazebo>
     <!-- Keel bulb -->
@@ -241,6 +249,7 @@
     </joint>
     <gazebo reference="rudder_joint">
-    </gazebo>
-    <!-- Mast -->
+        <provideFeedback>true</provideFeedback>
+    </gazebo>
+    <!-- Mast (visual only) -->
     <link name="mast_link">
         <visual>
@@ -283,5 +292,5 @@
     </link>
     <gazebo reference="main_sail_link">
-        <material>Gazebo/Gray</material>
+        <material>Gazebo/GreyTransparent</material>
     </gazebo>
     <joint name="main_sail_joint" type="revolute">
@@ -298,4 +307,5 @@
     </joint>
     <gazebo reference="main_sail_joint">
+        <provideFeedback>true</provideFeedback>
     </gazebo>
     <!-- Fore sail -->
@@ -320,5 +330,5 @@
     </link>
     <gazebo reference="fore_sail_link">
-        <material>Gazebo/Gray</material>
+        <material>Gazebo/GreyTransparent</material>
     </gazebo>
     <joint name="fore_sail_joint" type="revolute">
@@ -335,109 +345,11 @@
     </joint>
     <gazebo reference="fore_sail_joint">
-    </gazebo>
-    <!-- Camera -->
-    <!-- <link name="cam_link">
-        <visual>
-            <geometry>
-                <box size="${cam_size} ${cam_size} ${cam_size}"/>
-            </geometry>
-            <material name="red" />
-        </visual>
-        <collision>
-            <geometry>
-                <box size="${cam_size} ${cam_size} ${cam_size}"/>
-            </geometry>
-        </collision>
-        <xacro:solid_cuboid_inertial mass="${cam_mass}" x="${cam_size}" y="${cam_size}" z="${cam_size}" />
-    </link>
-    <joint name="cam_joint" type="fixed">
-        <axis xyz="0 1 0" />
-        <origin xyz="${hull_length/2 - 0.25} 0 ${hull_depth/2 + cam_size/2}" rpy="0 0 0"/>
-        <parent link="base_link"/>
-        <child link="cam_link"/>
-    </joint> -->
-    <!-- Ray -->
-    <!-- <link name="ray_link">
-        <visual>
-            <geometry>
-              <box size="${ray_size} ${ray_size} ${ray_size}"/>
-            </geometry>
-            <material name="red" />
-        </visual>
-        <collision>
-            <geometry>
-                <box size="${ray_size} ${ray_size} ${ray_size}"/>
-            </geometry>
-        </collision>
-        <xacro:solid_cuboid_inertial mass="${ray_mass}" x="${ray_size}" y="${ray_size}" z="${ray_size}" />
-    </link>
-    <joint name="ray_joint" type="fixed">
-        <axis xyz="0 1 0" />
-        <origin xyz="${hull_length/2 - 0.25} 0.4 ${hull_depth/2 + ray_size/2}" rpy="0 0 0"/>
-        <parent link="base_link"/>
-        <child link="ray_link"/>
-    </joint> -->
-    <!-- GPS -->
-    <!-- <link name="gps_link">
-        <visual>
-            <geometry>
-                <box size="${gps_size} ${gps_size} ${gps_size}"/>
-            </geometry>
-            <material name="red" />
-        </visual>
-        <collision>
-            <geometry>
-                <box size="${gps_size} ${gps_size} ${gps_size}"/>
-            </geometry>
-        </collision>
-        <xacro:solid_cuboid_inertial mass="${gps_mass}" x="${gps_size}" y="${gps_size}" z="${gps_size}" />
-    </link>
-    <joint name="gps_joint" type="fixed">
-        <axis xyz="0 1 0" />
-        <origin xyz="0 0.4 ${hull_depth/2 + gps_size/2}" rpy="0 0 0"/>
-        <parent link="base_link"/>
-        <child link="gps_link"/>
-    </joint> -->
-    <!-- IMU -->
-    <!-- <link name="imu_link">
-        <visual>
-            <geometry>
-                <box size="${imu_size} ${imu_size} ${imu_size}"/>
-            </geometry>
-            <material name="red" />
-        </visual>
-        <collision>
-            <geometry>
-                <box size="${imu_size} ${imu_size} ${imu_size}"/>
-            </geometry>
-        </collision>
-        <xacro:solid_cuboid_inertial mass="${imu_mass}" x="${imu_size}" y="${imu_size}" z="${imu_size}" />
-    </link>
-    <joint name="imu_joint" type="fixed">
-        <axis xyz="0 1 0" />
-        <origin xyz="0 0 ${hull_depth/2 + imu_size/2}" rpy="0 0 0"/>
-        <parent link="base_link"/>
-        <child link="imu_link"/>
-    </joint> -->
-    <!-- Magnetometer -->
-    <!-- <link name="mag_link">
-        <visual>
-            <geometry>
-                <box size="${mag_size} ${mag_size} ${mag_size}"/>
-            </geometry>
-            <material name="red" />
-        </visual>
-        <collision>
-            <geometry>
-                <box size="${mag_size} ${mag_size} ${mag_size}"/>
-            </geometry>
-        </collision>
-        <xacro:solid_cuboid_inertial mass="${gps_mass}" x="${mag_size}" y="${mag_size}" z="${mag_size}" />
-    </link>
-    <joint name="mag_joint" type="fixed">
-        <axis xyz="0 1 0" />
-        <origin xyz="0 -0.4 ${hull_depth/2 + mag_size/2}" rpy="0 0 0"/>
-        <parent link="base_link"/>
-        <child link="mag_link"/>
-    </joint> -->
+        <provideFeedback>true</provideFeedback>
+    </gazebo>
+    <!-- IMU  -->
+    <xacro:imu_link />
+    <xacro:imu_joint x="0.0" y="0.0" z="0.01" yaw="0" />
+    <!-- Anemometer (mast head) -->
+    <xacro:anemometer_link />
+    <xacro:anemometer_joint x="0.0" y="0.0" z="4.0" yaw="0" />
 </robot>

Commit message: Add positions controllers for rudder and sails
1. First version of controllers for rudder and sails using ros_control.
2. Add initial sketch of a hardware interface and configure position controllers.
3. Add rviz configuration for viewing the robot while being simulated.
4. Add gazebo elements for ros_control and transmission elements for joints.

File: rs750_description/urdf/rs750.urdf.xacro (robot description, xacro)
@@ -248,4 +248,13 @@
         <child link="rudder_link" />
     </joint>
+    <transmission name="rudder_transmission" >
+        <type>transmission_interface/SimpleTransmission</type>
+        <actuator name="rudder_actuator">
+            <mechanicalReduction>1</mechanicalReduction>
+        </actuator>
+        <joint name="rudder_joint">
+            <hardwareInterface>hardware_interface/PositionJointInterface</hardwareInterface>
+        </joint>
+    </transmission>
     <gazebo reference="rudder_joint">
         <provideFeedback>true</provideFeedback>
@@ -306,4 +315,13 @@
         <child link="main_sail_link" />
     </joint>
+    <transmission name="main_sail_transmission" >
+        <type>transmission_interface/SimpleTransmission</type>
+        <actuator name="main_sail_actuator">
+            <mechanicalReduction>1</mechanicalReduction>
+        </actuator>
+        <joint name="main_sail_joint">
+            <hardwareInterface>hardware_interface/PositionJointInterface</hardwareInterface>
+        </joint>
+    </transmission>
     <gazebo reference="main_sail_joint">
         <provideFeedback>true</provideFeedback>
@@ -344,4 +362,13 @@
         <child link="fore_sail_link" />
     </joint>
+    <transmission name="fore_sail_transmission" >
+        <type>transmission_interface/SimpleTransmission</type>
+        <actuator name="fore_sail_actuator">
+            <mechanicalReduction>1</mechanicalReduction>
+        </actuator>
+        <joint name="fore_sail_joint">
+            <hardwareInterface>hardware_interface/PositionJointInterface</hardwareInterface>
+        </joint>
+    </transmission>
     <gazebo reference="fore_sail_joint">
         <provideFeedback>true</provideFeedback>
@@ -350,6 +377,6 @@
     <xacro:imu_link />
     <xacro:imu_joint x="0.0" y="0.0" z="0.01" yaw="0" />
-    <!-- Anemometer (mast head) -->
-    <xacro:anemometer_link />
-    <xacro:anemometer_joint x="0.0" y="0.0" z="4.0" yaw="0" />
+    <!-- Anemometer (mast head) DISABLED - issue with plugin... -->
+    <!-- <xacro:anemometer_link />
+    <xacro:anemometer_joint x="0.0" y="0.0" z="4.0" yaw="0" /> -->
 </robot>

Commit message: Update robot description.
1. Separate out mag link.

File: rs750_description/urdf/rs750.urdf.xacro (robot description, xacro)
@@ -39,6 +39,7 @@
     <xacro:include filename="$(find rs750_description)/urdf/rs750_materials.xacro"/>
     <xacro:include filename="$(find rs750_description)/urdf/rs750_inertials.xacro"/>
+    <xacro:include filename="$(find rs750_description)/urdf/rs750_anemometer.xacro"/>
     <xacro:include filename="$(find rs750_description)/urdf/rs750_imu.xacro"/>
-    <xacro:include filename="$(find rs750_description)/urdf/rs750_anemometer.xacro"/>
+    <xacro:include filename="$(find rs750_description)/urdf/rs750_magnetic.xacro"/>
     <xacro:include filename="$(find rs750_description)/urdf/rs750.gazebo"/>
     <!-- Constants for robot dimensions -->
@@ -180,6 +181,6 @@
     <!-- Preserve fixed joint as the keel_fin_link has an associated plugin -->
     <gazebo reference="keel_fin_joint">
-        <disableFixedJointLumping>true</disableFixedJointLumping>
-        <preserveFixedJoint>true</preserveFixedJoint>
+        <!-- <disableFixedJointLumping>true</disableFixedJointLumping>  -->
+        <!-- <preserveFixedJoint>true</preserveFixedJoint> -->
     </gazebo>
     <!-- Keel bulb -->
@@ -374,9 +375,12 @@
         <provideFeedback>true</provideFeedback>
     </gazebo>
+    <!-- Anemometer (mast head) -->
+    <xacro:anemometer_link />
+    <xacro:anemometer_joint x="0.0" y="0.0" z="4.0" yaw="0" />
     <!-- IMU  -->
     <xacro:imu_link />
     <xacro:imu_joint x="0.0" y="0.0" z="0.01" yaw="0" />
-    <!-- Anemometer (mast head) -->
-    <xacro:anemometer_link />
-    <xacro:anemometer_joint x="0.0" y="0.0" z="4.0" yaw="0" />
+    <!-- IMU  -->
+    <xacro:magnetic_link />
+    <xacro:magnetic_joint x="0.0" y="0.0" z="0.01" yaw="0" />
 </robot>

File: rs750_description/urdf/rs750_anemometer.xacro (robot description, xacro)
@@ -33,5 +33,5 @@
 <robot xmlns:xacro="http://ros.org/wiki/xacro">
     <xacro:macro name="anemometer_link">
-        <link name="anemometer">
+        <link name="anemometer_link">
             <visual>
                 <origin rpy="0 0 0" xyz="0 0 0" />
@@ -50,5 +50,5 @@
                 mass="0.01" length="0.05" radius="0.02" />
         </link>
-        <gazebo reference="anemometer">
+        <gazebo reference="anemometer_link">
             <material>Gazebo/Green</material>
             <sensor type="anemometer" name="anemometer_sensor">
@@ -59,5 +59,5 @@
                 <plugin filename="libgazebo_ros_anemometer.so" name="anemometer_plugin">
                     <robotNamespace>/</robotNamespace>
-                    <frameId>anemometer</frameId>
+                    <frameId>anemometer_link</frameId>
                     <topicName>wind/apparent</topicName>
                 </plugin>
@@ -69,8 +69,8 @@
             <origin rpy="0 0 ${yaw}" xyz="${x} ${y} ${z}"/>
             <parent link="base_link" />
-            <child link="anemometer" />
+            <child link="anemometer_link" />
         </joint>
         <gazebo reference="anemometer_joint">
-            <preserveFixedJoint>true</preserveFixedJoint>
+            <!-- <preserveFixedJoint>true</preserveFixedJoint> -->
         </gazebo>
     </xacro:macro>

File: rs750_description/urdf/rs750_magnetic.xacro (robot description, xacro)
@@ -29,9 +29,9 @@
     POSSIBILITY OF SUCH DAMAGE.
 -->
-<!--  xacro macros for IMU sensor (dimensions for SparkFun BNO080).
+<!--  xacro macros for magnetic sensor (dimensions for SparkFun BNO080).
  -->
 <robot xmlns:xacro="http://ros.org/wiki/xacro">
-    <xacro:macro name="imu_link">
-        <link name="imu_link">
+    <xacro:macro name="magnetic_link">
+        <link name="magnetic_link">
             <visual>
                 <origin rpy="0 0 0" xyz="0 0 0" />
@@ -50,35 +50,34 @@
                 mass="0.004" x="0.031" y="0.026" z="0.005" />
         </link>
-        <gazebo reference="imu_link">
-            <material>Gazebo/Green</material>
-            <sensor type="imu" name="imu_sensor">
-                <always_on>true</always_on>
-                <update_rate>50</update_rate>
+        <!--
+        <gazebo reference="magnetic_link">
+            <sensor type="magnetometer" name="magnetic_sensor">
+                <always_on>1</always_on>>
+                <update_rate>100.0</update_rate>
                 <visualize>true</visualize>
-                <topic>sensors/imu</topic>
-                <pose>0 0 0 0 0 0</pose>
-                <imu>
-                    <topic>sensors/imu</topic>
-                </imu>
-                <plugin name="imu_plugin" filename="libgazebo_ros_imu_sensor.so">
-                    <gaussianNoise>0.0</gaussianNoise>
-                    <always_on>true</always_on>
-                    <updateRateHZ>50</updateRateHZ>
-                    <topicName>sensors/imu</topicName>
-                    <bodyName>imu_link</bodyName>
-                    <frameName>imu_link</frameName>
-                    <xyzOffset>0 0 0</xyzOffset>
-                    <rpyOffset>0 0 0</rpyOffset>
-                </plugin>
+                <magnetometer name="mag">
+                </magnetometer>
             </sensor>
         </gazebo>
+        -->
+        <gazebo>
+            <plugin name="magnetic_plugin" filename="libhector_gazebo_ros_magnetic.so">
+                <updateRate>10.0</updateRate>
+                <bodyName>magnetic_link</bodyName>
+                <frameId>magnetic_link</frameId>
+                <topicName>sensors/magnetic</topicName>
+                <offset>0 0 0</offset>
+                <drift>0.0 0.0 0.0</drift>
+                <gaussianNoise>1.3e-2 1.3e-2 1.3e-2</gaussianNoise>
+            </plugin>
+        </gazebo>
     </xacro:macro>
-    <xacro:macro name="imu_joint" params="x y z yaw" >
-        <joint name="imu_joint" type="fixed">
+    <xacro:macro name="magnetic_joint" params="x y z yaw" >
+        <joint name="magnetic_joint" type="fixed">
             <origin rpy="0 0 ${yaw}" xyz="${x} ${y} ${z}"/>
             <parent link="base_link" />
-            <child link="imu_link" />
+            <child link="magnetic_link" />
         </joint>
-        <gazebo reference="imu_joint">
+        <gazebo reference="magnetic_joint">
             <!-- <preserveFixedJoint>true</preserveFixedJoint> -->
         </gazebo>

Commit message: Update robot description
1. Refactor rs750 model, move rig into a separate xacro file.

File: rs750_description/urdf/rs750.urdf.xacro (robot description, xacro)
@@ -43,4 +43,5 @@
     <xacro:include filename="$(find rs750_description)/urdf/rs750_magnetic.xacro"/>
     <xacro:include filename="$(find rs750_description)/urdf/rs750.gazebo"/>
+    <xacro:include filename="$(find rs750_description)/urdf/rs750_rig.xacro"/>
     <!-- Constants for robot dimensions -->
     <xacro:property name="scale" value="3.2" />
@@ -261,118 +262,6 @@
         <provideFeedback>true</provideFeedback>
     </gazebo>
-    <!-- Mast (visual only) -->
-    <link name="mast_link">
-        <visual>
-            <origin rpy="0 0 0" xyz="0 0 0" />
-            <geometry>
-                <mesh filename="package://rs750_description/meshes/rs750_mast.stl" />
-            </geometry>
-            <material name="black" />
-        </visual>
-    </link>
-    <gazebo reference="mast_link">
-        <material>Gazebo/Black</material>
-    </gazebo>
-    <joint name="mast_joint" type="fixed">
-        <origin rpy="0 0 0" xyz="0 0 2.09"/>
-        <parent link="base_link" />
-        <child link="mast_link" />
-    </joint>
-    <gazebo reference="mast_joint">
-    </gazebo>
-    <!-- Main sail -->
-    <link name="main_sail_link">
-        <visual>
-            <origin rpy="0 0 0" xyz="0 0 0" />
-            <geometry>
-                <mesh filename="package://rs750_description/meshes/rs750_main_sail.stl" />
-            </geometry>
-            <material name="gray" />
-        </visual>
-        <collision>
-            <origin rpy="0 0 0" xyz="0 0 0" />
-            <geometry>
-                <mesh filename="package://rs750_description/meshes/rs750_main_sail.stl" />
-            </geometry>
-        </collision>
-        <xacro:solid_cuboid_inertial
-            rpy="0 0 0" xyz="0 0 0"
-            mass="${main_sail_mass}"
-            x="${main_sail_length}" y="${main_sail_width}" z="${main_sail_depth}" />
-    </link>
-    <gazebo reference="main_sail_link">
-        <material>Gazebo/GreyTransparent</material>
-    </gazebo>
-    <joint name="main_sail_joint" type="revolute">
-        <origin rpy="0 0 0" xyz="-0.02625 0 0.291875"/>
-        <axis xyz="0 0 1" />
-        <limit
-            lower="${-math_pi_over_2}"
-            upper="${math_pi_over_2}"
-            effort="1000"
-            velocity="1000"
-        />
-        <parent link="base_link" />
-        <child link="main_sail_link" />
-    </joint>
-    <transmission name="main_sail_transmission" >
-        <type>transmission_interface/SimpleTransmission</type>
-        <actuator name="main_sail_actuator">
-            <mechanicalReduction>1</mechanicalReduction>
-        </actuator>
-        <joint name="main_sail_joint">
-            <hardwareInterface>hardware_interface/PositionJointInterface</hardwareInterface>
-        </joint>
-    </transmission>
-    <gazebo reference="main_sail_joint">
-        <provideFeedback>true</provideFeedback>
-    </gazebo>
-    <!-- Fore sail -->
-    <link name="fore_sail_link">
-        <visual>
-            <origin rpy="0 0 0" xyz="0 0 0" />
-            <geometry>
-                <mesh filename="package://rs750_description/meshes/rs750_fore_sail.stl" />
-            </geometry>
-            <material name="gray" />
-        </visual>
-        <collision>
-            <origin rpy="0 0 0" xyz="0 0 0" />
-            <geometry>
-                <mesh filename="package://rs750_description/meshes/rs750_fore_sail.stl" />
-            </geometry>
-        </collision>
-        <xacro:solid_cuboid_inertial
-            rpy="0 0 0" xyz="0 0 0"
-            mass="${fore_sail_mass}"
-            x="${fore_sail_length}" y="${fore_sail_width}" z="${fore_sail_depth}" />
-    </link>
-    <gazebo reference="fore_sail_link">
-        <material>Gazebo/GreyTransparent</material>
-    </gazebo>
-    <joint name="fore_sail_joint" type="revolute">
-        <origin rpy="0 0 0" xyz="1.03125 0 0.235625"/>
-        <axis xyz="-0.271652766 0 0.962395332" />
-        <limit
-            lower="${-math_pi_over_2}"
-            upper="${math_pi_over_2}"
-            effort="1000"
-            velocity="1000"
-        />
-        <parent link="base_link" />
-        <child link="fore_sail_link" />
-    </joint>
-    <transmission name="fore_sail_transmission" >
-        <type>transmission_interface/SimpleTransmission</type>
-        <actuator name="fore_sail_actuator">
-            <mechanicalReduction>1</mechanicalReduction>
-        </actuator>
-        <joint name="fore_sail_joint">
-            <hardwareInterface>hardware_interface/PositionJointInterface</hardwareInterface>
-        </joint>
-    </transmission>
-    <gazebo reference="fore_sail_joint">
-        <provideFeedback>true</provideFeedback>
-    </gazebo>
+    <!-- Rig -->
+    <xacro:rig base_link="base_link" x="0.0" y="0.0" z="0.0"/>
     <!-- Anemometer (mast head) -->
     <xacro:anemometer_link />
