Commit message: Add a model for testing sail control.
1. Add a model containing just the rig to test sail controllers
2. Add a simple sail controller
3. Move the twist_translate node into the controllers package.

File: rs750_description/urdf/rs750.urdf.xacro (robot description, xacro)
@@ -42,6 +42,6 @@
     <xacro:include filename="$(find rs750_description)/urdf/rs750_imu.xacro"/>
     <xacro:include filename="$(find rs750_description)/urdf/rs750_magnetic.xacro"/>
+    <xacro:include filename="$(find rs750_description)/urdf/rs750_rig.xacro"/>
     <xacro:include filename="$(find rs750_description)/urdf/rs750.gazebo"/>
-    <xacro:include filename="$(find rs750_description)/urdf/rs750_rig.xacro"/>
     <!-- Constants for robot dimensions -->
     <xacro:property name="scale" value="3.2" />
@@ -111,5 +111,5 @@
             <material name="red" />
         </visual>
-        <collision name="hull_collision">
+        <collision>
             <origin rpy="0 0 0" xyz="0 0 0" />
             <geometry>
@@ -263,5 +263,5 @@
     </gazebo>
     <!-- Rig -->
-    <xacro:rig base_link="base_link" x="0.0" y="0.0" z="0.0"/>
+    <xacro:rig base_link="base_link" scale="${scale}" x="0.0" y="0.0" z="0.0"/>
     <!-- Anemometer (mast head) -->
     <xacro:anemometer_link />
@@ -270,5 +270,5 @@
     <xacro:imu_link />
     <xacro:imu_joint x="0.0" y="0.0" z="0.01" yaw="0" />
-    <!-- IMU  -->
+    <!-- Magnetometer  -->
     <xacro:magnetic_link />
     <xacro:magnetic_joint x="0.0" y="0.0" z="0.01" yaw="0" />

File: rs750_description/urdf/rs750_rig.xacro (robot description, xacro)
@@ -32,5 +32,15 @@
  -->
 <robot xmlns:xacro="http://ros.org/wiki/xacro">
-    <xacro:macro name="rig" params="base_link x y z">
+    <xacro:macro name="rig" params="base_link scale x y z">
+        <!-- Rough estimates for intertial -->
+        <xacro:property name="main_sail_mass" value="${0.100 * scale * scale * scale}" />
+        <xacro:property name="main_sail_length" value="${0.200 * scale}" />
+        <xacro:property name="main_sail_width" value="${0.006 * scale}" />
+        <xacro:property name="main_sail_depth" value="${0.900 * scale}" />
+        <!-- Rough estimates for intertial -->
+        <xacro:property name="fore_sail_mass" value="${0.0500 * scale * scale * scale}" />
+        <xacro:property name="fore_sail_length" value="${0.100 * scale}" />
+        <xacro:property name="fore_sail_width" value="${0.006 * scale}" />
+        <xacro:property name="fore_sail_depth" value="${0.700 * scale}" />
         <!-- Mast (visual only) -->
         <link name="mast_link">
